Commit message: feat：添加底盘的物理惯性属性

File: mrobot_desc_ws/src/mrobot_description/urdf/mrobot_chassis.urdf (robot description, URDF)
Before this commit: robot mrobot_chassis, 6 links, 5 joints
Links:
- link base_link: mass None -> 2; geometry collision cylinder length=0.005 radius=0.13; visual cylinder length=0.005 radius=0.13
